File: pcb/rp2040-programmer-calculator/buttons.kicad_sch (KiCad schematic)
At the start: 64 parts, among them SW1 PTS636SL50 LFS, SW10 PTS636SL50 LFS, SW11 PTS636SL50 LFS, SW12 PTS636SL50 LFS, SW13 PTS636SL50 LFS, SW14 PTS636SL50 LFS, SW15 PTS636SL50 LFS, SW16 PTS636SL50 LFS, SW17 PTS636SL50 LFS, SW18 PTS636SL50 LFS, SW19 PTS636SL50 LFS, SW2 PTS636SL50 LFS, SW20 PTS636SL50 LFS, SW21 PTS636SL50 LFS, SW22 PTS636SL50 LFS, SW23 PTS636SL50 LFS, SW24 PTS636SL50 LFS, SW25 PTS636SL50 LFS, SW26 PTS636SL50 LFS, SW27 PTS636SL50 LFS, SW28 PTS636SL50 LFS, SW29 PTS636SL50 LFS, SW3 PTS636SL50 LFS, SW30 PTS636SL50 LFS, SW31 PTS636SL50 LFS, SW32 PTS636SL50 LFS, SW4 PTS636SL50 LFS, SW5 PTS636SL50 LFS, SW6 PTS636SL50 LFS, SW7 PTS636SL50 LFS, SW8 PTS636SL50 LFS, SW9 PTS636SL50 LFS

Commit message: Finish PCB
Parts:
- renumbered D6 to D10, D10 to D11, D14 to D12, D18 to D13, D22 to D14, D26 to D15, D30 to D16, D3 to D17, D7 to D18, D11 to D19, D5 to D2, D15 to D20, D19 to D21, D23 to D22, D27 to D23, D31 to D24, D4 to D25, D8 to D26, D12 to D27, D16 to D28, D20 to D29, D9 to D3, D24 to D30, D28 to D31, D13 to D4, D17 to D5, D21 to D6, D25 to D7, D29 to D8, D2 to D9, SW2 to SW10, SW6 to SW11, SW10 to SW12, SW14 to SW13, SW18 to SW14, SW22 to SW15, SW26 to SW16, SW30 to SW17, SW3 to SW18, SW7 to SW19, SW1 to SW2, SW11 to SW20, SW15 to SW21, SW19 to SW22, SW27 to SW24, SW31 to SW25, SW4 to SW26, SW8 to SW27, SW12 to SW28, SW16 to SW29, SW5 to SW3, SW20 to SW30, SW24 to SW31, SW28 to SW32, SW32 to SW33, SW9 to SW4, SW13 to SW5, SW17 to SW6, SW21 to SW7, SW25 to SW8, SW29 to SW9

Commit message: Finished design
Parts:
- SW10, SW11, SW12, SW13, SW14, SW15, SW16, SW17, SW18, SW19, SW2, SW20, SW21, SW22, SW23, SW24, SW25, SW26, SW27, SW28, SW29, SW3, SW30, SW31, SW32, SW33, SW4, SW5, SW6, SW7, SW8, SW9: footprint SamacSys_Parts:PTS636SL50LFS -> PTS636SL50LFS:PTS636SL50LFS
Changed lines of the file:
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@@
 (kicad_sch
-	(version 20231120)
+	(version 20250114)
 	(generator "eeschema")
-	(generator_version "8.0")
+	(generator_version "9.0")
 	(paper "A4")
 	(junction
@@
 			)
 		)
-		(property "Footprint" "SamacSys_Parts:PTS636SL50LFS"
+		(property "Footprint" "PTS636SL50LFS:PTS636SL50LFS"
 			(at 82.55 58.42 0)
 			(effects
@@
 			)
 		)
-		(property "Footprint" "SamacSys_Parts:PTS636SL50LFS"
+		(property "Footprint" "PTS636SL50LFS:PTS636SL50LFS"
 			(at 82.55 96.52 0)
 			(effects
@@
 			)
 		)
-		(property "Footprint" "SamacSys_Parts:PTS636SL50LFS"
+		(property "Footprint" "PTS636SL50LFS:PTS636SL50LFS"
 			(at 57.15 83.82 0)
 			(effects
@@
 			)
 		)
-		(property "Footprint" "SamacSys_Parts:PTS636SL50LFS"
+		(property "Footprint" "PTS636SL50LFS:PTS636SL50LFS"
 			(at 133.35 109.22 0)
 			(effects
@@
 			)
 		)
-		(property "Footprint" "SamacSys_Parts:PTS636SL50LFS"
+		(property "Footprint" "PTS636SL50LFS:PTS636SL50LFS"
 			(at 133.35 96.52 0)
 			(effects
@@
 			)
 		)
-		(property "Footprint" "SamacSys_Parts:PTS636SL50LFS"
+		(property "Footprint" "PTS636SL50LFS:PTS636SL50LFS"
 			(at 107.95 58.42 0)
 			(effects
@@
 			)
 		)
-		(property "Footprint" "SamacSys_Parts:PTS636SL50LFS"
+		(property "Footprint" "PTS636SL50LFS:PTS636SL50LFS"
 			(at 82.55 33.02 0)
 			(effects
@@
 			)
 		)
-		(property "Footprint" "SamacSys_Parts:PTS636SL50LFS"
+		(property "Footprint" "PTS636SL50LFS:PTS636SL50LFS"
 			(at 133.35 58.42 0)
 			(effects
@@
 			)
 		)
-		(property "Footprint" "SamacSys_Parts:PTS636SL50LFS"
+		(property "Footprint" "PTS636SL50LFS:PTS636SL50LFS"
 			(at 82.55 109.22 0)
 			(effects
@@
 			)
 		)
-		(property "Footprint" "SamacSys_Parts:PTS636SL50LFS"
+		(property "Footprint" "PTS636SL50LFS:PTS636SL50LFS"
 			(at 57.15 96.52 0)
 			(effects
@@
 			)
 		)
-		(property "Footprint" "SamacSys_Parts:PTS636SL50LFS"
+		(property "Footprint" "PTS636SL50LFS:PTS636SL50LFS"
 			(at 107.95 109.22 0)
 			(effects
@@
 			)
 		)
-		(property "Footprint" "SamacSys_Parts:PTS636SL50LFS"
+		(property "Footprint" "PTS636SL50LFS:PTS636SL50LFS"
 			(at 133.35 121.92 0)
 			(effects
@@
 			)
 		)
-		(property "Footprint" "SamacSys_Parts:PTS636SL50LFS"
+		(property "Footprint" "PTS636SL50LFS:PTS636SL50LFS"
 			(at 57.15 121.92 0)
 			(effects
@@
 			)
 		)
-		(property "Footprint" "SamacSys_Parts:PTS636SL50LFS"
+		(property "Footprint" "PTS636SL50LFS:PTS636SL50LFS"
 			(at 82.55 121.92 0)
 			(effects
@@
 			)
 		)
-		(property "Footprint" "SamacSys_Parts:PTS636SL50LFS"
+		(property "Footprint" "PTS636SL50LFS:PTS636SL50LFS"
 			(at 82.55 45.72 0)
 			(effects
@@
 			)
 		)
-		(property "Footprint" "SamacSys_Parts:PTS636SL50LFS"
+		(property "Footprint" "PTS636SL50LFS:PTS636SL50LFS"
 			(at 133.35 33.02 0)
 			(effects
@@
 			)
 		)
-		(property "Footprint" "SamacSys_Parts:PTS636SL50LFS"
+		(property "Footprint" "PTS636SL50LFS:PTS636SL50LFS"
 			(at 57.15 71.12 0)
 			(effects
@@
 			)
 		)
-		(property "Footprint" "SamacSys_Parts:PTS636SL50LFS"
+		(property "Footprint" "PTS636SL50LFS:PTS636SL50LFS"
 			(at 82.55 71.12 0)
 			(effects
@@
 			)
 		)
-		(property "Footprint" "SamacSys_Parts:PTS636SL50LFS"
+		(property "Footprint" "PTS636SL50LFS:PTS636SL50LFS"
 			(at 107.95 83.82 0)
 			(effects
@@
 			)
 		)
-		(property "Footprint" "SamacSys_Parts:PTS636SL50LFS"
+		(property "Footprint" "PTS636SL50LFS:PTS636SL50LFS"
 			(at 133.35 83.82 0)
 			(effects
@@
 			)
 		)
-		(property "Footprint" "SamacSys_Parts:PTS636SL50LFS"
+		(property "Footprint" "PTS636SL50LFS:PTS636SL50LFS"
 			(at 57.15 33.02 0)
 			(effects
@@
 			)
 		)
-		(property "Footprint" "SamacSys_Parts:PTS636SL50LFS"
+		(property "Footprint" "PTS636SL50LFS:PTS636SL50LFS"
 			(at 107.95 96.52 0)
 			(effects
@@
 			)
 		)
-		(property "Footprint" "SamacSys_Parts:PTS636SL50LFS"
+		(property "Footprint" "PTS636SL50LFS:PTS636SL50LFS"
 			(at 57.15 58.42 0)
 			(effects
@@
 			)
 		)
-		(property "Footprint" "SamacSys_Parts:PTS636SL50LFS"
+		(property "Footprint" "PTS636SL50LFS:PTS636SL50LFS"
 			(at 82.55 83.82 0)
 			(effects
@@
 			)
 		)
-		(property "Footprint" "SamacSys_Parts:PTS636SL50LFS"
+		(property "Footprint" "PTS636SL50LFS:PTS636SL50LFS"
 			(at 107.95 33.02 0)
 			(effects
@@
 			)
 		)
-		(property "Footprint" "SamacSys_Parts:PTS636SL50LFS"
+		(property "Footprint" "PTS636SL50LFS:PTS636SL50LFS"
 			(at 107.95 71.12 0)
 			(effects
@@
 			)
 		)
-		(property "Footprint" "SamacSys_Parts:PTS636SL50LFS"
+		(property "Footprint" "PTS636SL50LFS:PTS636SL50LFS"
 			(at 107.95 45.72 0)
 			(effects
@@
 			)
 		)
-		(property "Footprint" "SamacSys_Parts:PTS636SL50LFS"
+		(property "Footprint" "PTS636SL50LFS:PTS636SL50LFS"
 			(at 57.15 45.72 0)
 			(effects
@@
 			)
 		)
-		(property "Footprint" "SamacSys_Parts:PTS636SL50LFS"
+		(property "Footprint" "PTS636SL50LFS:PTS636SL50LFS"
 			(at 57.15 109.22 0)
 			(effects
@@
 			)
 		)
-		(property "Footprint" "SamacSys_Parts:PTS636SL50LFS"
+		(property "Footprint" "PTS636SL50LFS:PTS636SL50LFS"
 			(at 107.95 121.92 0)
 			(effects
@@
 			)
 		)
-		(property "Footprint" "SamacSys_Parts:PTS636SL50LFS"
+		(property "Footprint" "PTS636SL50LFS:PTS636SL50LFS"
 			(at 133.35 71.12 0)
 			(effects
@@
 			)
 		)
-		(property "Footprint" "SamacSys_Parts:PTS636SL50LFS"
+		(property "Footprint" "PTS636SL50LFS:PTS636SL50LFS"
 			(at 133.35 45.72 0)
 			(effects
