File: pcb/rp2040-programmer-calculator/keys.kicad_sch (KiCad schematic)
At the start: 60 parts, among them SW33 B3F, SW34 B3F, SW35 B3F, SW36 B3F, SW37 B3F, SW38 B3F, SW39 B3F, SW40 B3F, SW41 B3F, SW42 B3F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

Commit message: Finish PCB
Parts:
- renumbered SW33 to SW34, SW34 to SW35, SW35 to SW36, SW36 to SW37, SW37 to SW38, SW38 to SW39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
