File: pcb/rp2040-programmer-calculator/led_byte.kicad_sch (KiCad schematic)
At the start: 18 parts, among them U3 74HC595

Commit message: Finish PCB
Parts:
- C5: renamed from C2; footprint (none) -> Capacitor_SMD:C_0603_1608Metric
- R16: renamed from R11; footprint (none) -> Resistor_SMD:R_0603_1608Metric_Pad0.98x0.95mm_HandSolder
- R17: renamed from R5; footprint (none) -> Resistor_SMD:R_0603_1608Metric_Pad0.98x0.95mm_HandSolder
- R18: renamed from R10; footprint (none) -> Resistor_SMD:R_0603_1608Metric_Pad0.98x0.95mm_HandSolder
- R19: renamed from R12; footprint (none) -> Resistor_SMD:R_0603_1608Metric_Pad0.98x0.95mm_HandSolder
- R20, R21: footprint (none) -> Resistor_SMD:R_0603_1608Metric_Pad0.98x0.95mm_HandSolder
- R22: renamed from R29; footprint (none) -> Resistor_SMD:R_0603_1608Metric_Pad0.98x0.95mm_HandSolder
- R23: renamed from R30; footprint (none) -> Resistor_SMD:R_0603_1608Metric_Pad0.98x0.95mm_HandSolder
- renumbered D63 to D71, D64 to D72, D65 to D73, D66 to D74, D67 to D75, D68 to D76, D69 to D77, D70 to D78, U3 to U4
Connections:
- net GND: now also D71.1 (K), D72.1 (K), D73.1 (K), D74.1 (K), D75.1 (K), D76.1 (K), D77.1 (K), D78.1 (K); no longer R16.2, R17.2, R18.2, R19.2, R20.2, R21.2, R22.2, R23.2
- net at R21.1: now also U4.5 (QF); no longer D76.1 (K)
- net at D76.2 (A): now also R21.2; no longer U4.5 (QF)
- net at R22.1: now also U4.6 (QG); no longer D77.1 (K)
- net at R19.1: now also U4.3 (QD); no longer D74.1 (K)
- net at R16.1: now also U4.15 (QA); no longer D71.1 (K)
- net at D71.2 (A): now also R16.2; no longer U4.15 (QA)
- net at D77.2 (A): now also R22.2; no longer U4.6 (QG)
- net at R18.1: now also U4.2 (QC); no longer D73.1 (K)
- net at R23.1: now also U4.7 (QH); no longer D78.1 (K)
- net at R20.1: now also U4.4 (QE); no longer D75.1 (K)
- net at U4.1 (QB): now also R17.1; no longer D72.2 (A)
- net at D73.2 (A): now also R18.2; no longer U4.2 (QC)
- net at D74.2 (A): now also R19.2; no longer U4.3 (QD)
- net at D75.2 (A): now also R20.2; no longer U4.4 (QE)
- net at D78.2 (A): now also R23.2; no longer U4.7 (QH)
- new net: D72.2 (A), R17.2
Other:
- moved on the sheet: D71, D72, D73, D74, D75, D76, D77, D78, R16, R17, R18, R19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

Commit message: Finished design
Parts:
- renumbered C5 to C4, D71 to D63, D72 to D64, D73 to D65, D74 to D66, D75 to D67, D76 to D68, D77 to D69, D78 to D70, R18 to R10, R19 to R11, R20 to R12, R21 to R13, R22 to R14, R23 to R15, R16 to R8, R17 to R9, U4 to U3
Connections:
- net at R14.1: now also U3.1 (QB); no longer U3.6 (QG)
- net at R11.1: now also U3.4 (QE); no longer U3.3 (QD)
- net at R8.1: now also U3.7 (QH); no longer U3.15 (QA)
- net at R10.1: now also U3.5 (QF); no longer U3.2 (QC)
- net at R15.1: now also U3.15 (QA); no longer U3.7 (QH)
- net at R12.1: now also U3.3 (QD); no longer U3.4 (QE)
- net at R9.1: now also U3.6 (QG); no longer U3.1 (QB)
- net at R13.1: now also U3.2 (QC); no longer U3.5 (QF)
Other:
- moved on the sheet: D63, D64, D65, D66, D67, D68, D69, D70, R10, R11, R12, R13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
