File: pcb/rp2040-programmer-calculator/matrix.kicad_sch (KiCad schematic)
At the start: 4 parts, among them U1 TCA8418RTWR

Commit message: Finish PCB
Parts:
- C3: renamed from C1; footprint (none) -> Capacitor_SMD:C_0402_1005Metric
- R6: renamed from R1; footprint (none) -> Resistor_SMD:R_0603_1608Metric
- R7: renamed from R2; footprint (none) -> Resistor_SMD:R_0603_1608Metric
- U2: renamed from U1; footprint TCA8418RTWR:QFN50P400X400X80-25N -> TCA8418RWTR:QFN50P400X400X80-25N
Changed lines of the file:
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@@
 		(dnp no)
 		(fields_autoplaced yes)
-		(property "Reference" "C1"
+		(property "Reference" "C3"
 			(at 69.85 26.6699 0)
 			(effects
@@
 			)
 		)
-		(property "Footprint" ""
+		(property "Footprint" "Capacitor_SMD:C_0402_1005Metric"
 			(at 67.0052 31.75 0)
 			(effects
@@
 			(project ""
 				(path "/a76e07d4-0b9a-412a-8673-6db50899653e/f05d4cfd-525d-48e4-b658-a76a5d301532"
-					(reference "C1")
+					(reference "C3")
 					(unit 1)
 				)
@@
 		(dnp no)
 		(fields_autoplaced yes)
-		(property "Reference" "#PWR01"
+		(property "Reference" "#PWR016"
 			(at 99.06 109.22 0)
 			(effects
@@
 			(project ""
 				(path "/a76e07d4-0b9a-412a-8673-6db50899653e/f05d4cfd-525d-48e4-b658-a76a5d301532"
-					(reference "#PWR01")
+					(reference "#PWR016")
 					(unit 1)
 				)
@@
 		(dnp no)
 		(fields_autoplaced yes)
-		(property "Reference" "#PWR03"
+		(property "Reference" "#PWR013"
 			(at 66.04 40.64 0)
 			(effects
@@
 			(project ""
 				(path "/a76e07d4-0b9a-412a-8673-6db50899653e/f05d4cfd-525d-48e4-b658-a76a5d301532"
-					(reference "#PWR03")
+					(reference "#PWR013")
 					(unit 1)
 				)
@@
 		(dnp no)
 		(fields_autoplaced yes)
-		(property "Reference" "#PWR02"
+		(property "Reference" "#PWR012"
 			(at 58.42 22.86 0)
 			(effects
@@
 			(project ""
 				(path "/a76e07d4-0b9a-412a-8673-6db50899653e/f05d4cfd-525d-48e4-b658-a76a5d301532"
-					(reference "#PWR02")
+					(reference "#PWR012")
 					(unit 1)
 				)
@@
 		(dnp no)
 		(fields_autoplaced yes)
-		(property "Reference" "R1"
+		(property "Reference" "R6"
 			(at 49.53 46.9899 0)
 			(effects
@@
 			)
 		)
-		(property "Footprint" ""
+		(property "Footprint" "Resistor_SMD:R_0603_1608Metric"
 			(at 48.006 48.514 90)
 			(effects
@@
 			(project ""
 				(path "/a76e07d4-0b9a-412a-8673-6db50899653e/f05d4cfd-525d-48e4-b658-a76a5d301532"
-					(reference "R1")
+					(reference "R6")
 					(unit 1)
 				)
@@
 		(dnp no)
 		(fields_autoplaced yes)
-		(property "Reference" "U1"
+		(property "Reference" "U2"
 			(at 78.74 39.37 0)
 			(effects
@@
 			)
 		)
-		(property "Footprint" "TCA8418RTWR:QFN50P400X400X80-25N"
+		(property "Footprint" "TCA8418RWTR:QFN50P400X400X80-25N"
 			(at 78.74 72.39 0)
 			(effects
@@
 			(project ""
 				(path "/a76e07d4-0b9a-412a-8673-6db50899653e/f05d4cfd-525d-48e4-b658-a76a5d301532"
-					(reference "U1")
+					(reference "U2")
 					(unit 1)
 				)
@@
 		(dnp no)
 		(fields_autoplaced yes)
-		(property "Reference" "#PWR05"
+		(property "Reference" "#PWR015"
 			(at 104.14 45.72 0)
 			(effects
@@
 			(project "rp2040-programmer-calculator"
 				(path "/a76e07d4-0b9a-412a-8673-6db50899653e/f05d4cfd-525d-48e4-b658-a76a5d301532"
-					(reference "#PWR05")
+					(reference "#PWR015")
 					(unit 1)
 				)
@@
 		(dnp no)
 		(fields_autoplaced yes)
-		(property "Reference" "#PWR04"
+		(property "Reference" "#PWR014"
 			(at 46.99 45.72 0)
 			(effects
@@
 			(project ""
 				(path "/a76e07d4-0b9a-412a-8673-6db50899653e/f05d4cfd-525d-48e4-b658-a76a5d301532"
-					(reference "#PWR04")
+					(reference "#PWR014")
 					(unit 1)
 				)
@@
 		(dnp no)
 		(fields_autoplaced yes)
-		(property "Reference" "R2"
+		(property "Reference" "R7"
 			(at 106.68 46.9899 0)
 			(effects
@@
 			)
 		)
-		(property "Footprint" ""
+		(property "Footprint" "Resistor_SMD:R_0603_1608Metric"
 			(at 105.156 48.514 90)
 			(effects
@@
 			(project "rp2040-programmer-calculator"
 				(path "/a76e07d4-0b9a-412a-8673-6db50899653e/f05d4cfd-525d-48e4-b658-a76a5d301532"
-					(reference "R2")
-					(unit 1)
-				)
+					(reference "R7")
+					(unit 1)
+				)

Commit message: Finished design
Parts:
- C3: footprint Capacitor_SMD:C_0402_1005Metric -> Capacitor_SMD:C_0603_1608Metric
- U2: footprint TCA8418RWTR:QFN50P400X400X80-25N -> TCA8418RTWR:QFN50P400X400X80-25N
Changed lines of the file:
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@@
 (kicad_sch
-	(version 20231120)
+	(version 20250114)
 	(generator "eeschema")
-	(generator_version "8.0")
+	(generator_version "9.0")
 	(paper "A4")
 	(junction
@@
 			)
 		)
-		(property "Footprint" "Capacitor_SMD:C_0402_1005Metric"
+		(property "Footprint" "Capacitor_SMD:C_0603_1608Metric"
 			(at 67.0052 31.75 0)
 			(effects
@@
 			)
 		)
-		(property "Footprint" "TCA8418RWTR:QFN50P400X400X80-25N"
+		(property "Footprint" "TCA8418RTWR:QFN50P400X400X80-25N"
 			(at 78.74 72.39 0)
 			(effects
@@
 		(at 143.51 57.15)
 		(size 21.59 25.4)
+		(exclude_from_sim no)
+		(in_bom yes)
+		(on_board yes)
+		(dnp no)
 		(stroke
 			(width 0.1524)
@@
 		(at 143.51 95.25)
 		(size 21.59 30.48)
+		(exclude_from_sim no)
+		(in_bom yes)
+		(on_board yes)
+		(dnp no)
 		(stroke
 			(width 0.1524)
