File: pcb/rp2040-programmer-calculator/rp2040-programmer-calculator.kicad_sch (KiCad schematic)
At the start: 7 parts, among them U2 RP2040, Y1 ABM8-272-T3

Commit message: Finish schematic
Parts:
- added J2: 5*2.54mm DNP, symbol Connector_Generic:Conn_01x05
- added R56, R57: 4.7k, symbol Device:R_US
- added SW64: PTS636SL50 LFS, SamacSys_Parts:PTS636SL50LFS, symbol Switch:SW_Push
- added TP10: GPIO28, symbol Connector:TestPoint
- added TP11: GPIO27, symbol Connector:TestPoint
- added TP12: GPIO11, symbol Connector:TestPoint
- added TP13: GPIO12, symbol Connector:TestPoint
- added TP8: ~{STDBY}, symbol Connector:TestPoint
- added TP9: GPIO29, symbol Connector:TestPoint
Connections:
- net +3V3: now also J2.5 (Pin_5), R56.2, R57.2
- net GND: now also J2.3 (Pin_3), SW64.1
- net LED_RCLK: now also U2.28 (GPIO17)
- net LED_SER: now also U2.18 (GPIO15)
- net LED_SRCLK: now also U2.17 (GPIO14)
- net LED_~{OE}: now also U2.29 (GPIO18)
- net LED_~{SRCLR}: now also U2.27 (GPIO16)
- net MATRIX_I2C_SCL: now also U2.3 (GPIO1), R56.1
- net MATRIX_I2C_SDA: now also U2.2 (GPIO0), R57.1
- net MATRIX_~{INT}: now also U2.5 (GPIO3)
- net MATRIX_~{RESET}: now also U2.4 (GPIO2)
- net RUN: now also J2.1 (Pin_1), SW64.2
- net SWCLK: now also J2.4 (Pin_4)
- net SWD: now also J2.2 (Pin_2)
- net LCD_D/~{C}: now reaches U2.11 (GPIO8)
- net LCD_~{RESET}: now reaches U2.12 (GPIO9)
- net at U2.14 (GPIO11): now also TP12.1
- net at U2.15 (GPIO12): now also TP13.1
- net ~{CHRG}: now reaches U2.31 (GPIO20)
- net PWR_EN: now reaches U2.34 (GPIO22)
- net PWR_BTN: now reaches U2.35 (GPIO23)
- net BAT_ADC_EN: now reaches U2.37 (GPIO25)
- net BAT_ADC: now reaches U2.38 (GPIO26_ADC0)
- net at U2.39 (GPIO27_ADC1): now also TP11.1
- net at U2.40 (GPIO28_ADC2): now also TP10.1
- net at U2.41 (GPIO29_ADC3): now also TP9.1
- net LCD_SPI_~{CS}: now reaches U2.7 (GPIO5)
- net LCD_SPI_CLK: now reaches U2.8 (GPIO6)
- net LCD_SPI_DIN: now reaches U2.9 (GPIO7)
- new net Power/~{STDBY}: TP8.1
- no-connect marks 0 -> 5
Other:
- added sheet Display (display.kicad_sch)
- sheet Power ports: added BAT_ADC, BAT_ADC_EN, PWR_BTN, PWR_EN, ~{CHRG}, ~{STDBY}; removed none
- note added: "Debug header"
- note added: "I2C pullups 0603 so easily swappable"
- note added: "on SPI pins in case we want to drive that way"
- moved on the sheet: C6, C7, R35, R41, R42, U2, Y1

Commit message: Finish PCB
Parts:
- J1: renamed from J2; footprint (none) -> Connector_PinHeader_2.54mm:PinHeader_1x05_P2.54mm_Vertical
- R1: renamed from R56; footprint (none) -> Resistor_SMD:R_0603_1608Metric
- R2: renamed from R57; footprint (none) -> Resistor_SMD:R_0603_1608Metric
- R3: renamed from R42; footprint (none) -> Resistor_SMD:R_0402_1005Metric
- R4: renamed from R41; footprint (none) -> Resistor_SMD:R_0402_1005Metric
- R5: renamed from R35; footprint (none) -> Resistor_SMD:R_0402_1005Metric
- TP1: renamed from TP8; footprint (none) -> TestPoint:TestPoint_Pad_D1.0mm
- TP2: renamed from TP12; footprint (none) -> TestPoint:TestPoint_Pad_D1.0mm
- TP3: renamed from TP13; footprint (none) -> TestPoint:TestPoint_Pad_D1.0mm
- TP4: renamed from TP11; footprint (none) -> TestPoint:TestPoint_Pad_D1.0mm
- TP5: renamed from TP10; footprint (none) -> TestPoint:TestPoint_Pad_D1.0mm
- TP6: renamed from TP9; footprint (none) -> TestPoint:TestPoint_Pad_D1.0mm
- renumbered C6 to C1, C7 to C2, SW64 to SW1, U2 to U1
Connections:
- net MATRIX_~{INT}: now also U1.4 (GPIO2); no longer U1.5 (GPIO3)
- net MATRIX_~{RESET}: now also U1.5 (GPIO3); no longer U1.4 (GPIO2)
- net USB/USB_DM renamed USB/USB_DN
- no-connect marks 5 -> 6
Other:
- sheet USB ports: added USB_DN; removed USB_DM

Commit message: Finished design
Parts:
- removed TP1: ~{STDBY}, TestPoint:TestPoint_Pad_D1.0mm, symbol Connector:TestPoint
- removed TP2: GPIO11, TestPoint:TestPoint_Pad_D1.0mm, symbol Connector:TestPoint
- removed TP3: GPIO12, TestPoint:TestPoint_Pad_D1.0mm, symbol Connector:TestPoint
- removed TP4: GPIO27, TestPoint:TestPoint_Pad_D1.0mm, symbol Connector:TestPoint
- removed TP5: GPIO28, TestPoint:TestPoint_Pad_D1.0mm, symbol Connector:TestPoint
- removed TP6: GPIO29, TestPoint:TestPoint_Pad_D1.0mm, symbol Connector:TestPoint
- added J3: Spare GPIO, Connector_PinHeader_2.00mm:PinHeader_1x03_P2.00mm_Vertical, symbol Connector_Generic:Conn_01x03
- SW1: value PTS636SL50 LFS -> PTS815_SJM_250_SMTR_LFS; footprint SamacSys_Parts:PTS636SL50LFS -> PTS815_SJM_250_SMTR_LFS:SW_Push_PTS815_SJM_250_SMTR_LFS
Connections:
- net at U1.39 (GPIO27_ADC1): now also J3.1 (Pin_1)
- net at U1.41 (GPIO29_ADC3): now also J3.3 (Pin_3)
- net at U1.40 (GPIO28_ADC2): now also J3.2 (Pin_2)
- net ~{STDBY}: now reaches U1.30 (GPIO19)
- no-connect marks 6 -> 7
