File: pcb/rp2040-programmer-calculator/usb.kicad_sch (KiCad schematic)
At the start: 3 parts, among them J1 USB4105-GF-A

Commit message: Finish PCB
Parts:
- removed R39: 5.1k, symbol Device:R_US
- added R43: 5.1k, Resistor_SMD:R_0603_1608Metric, symbol Device:R_US
- R42: renamed from R38; footprint (none) -> Resistor_SMD:R_0603_1608Metric
- renumbered J1 to J2
Connections:
- net GND: now also R43.2
- net at J2.B5 (CC2): now also R43.1
- net USB_DM renamed USB_DN
Changed lines of the file:
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@@
 		)
 	)
-	(hierarchical_label "USB_DM"
+	(hierarchical_label "USB_DN"
 		(shape input)
 		(at 114.3 83.82 0)
@@
 		(dnp no)
 		(fields_autoplaced yes)
-		(property "Reference" "#PWR032"
+		(property "Reference" "#PWR038"
 			(at 85.09 119.38 0)
 			(effects
@@
 			(project "rp2040-programmer-calculator"
 				(path "/a76e07d4-0b9a-412a-8673-6db50899653e/0f3726b0-757f-41d2-86b9-fa06e0efb2c9"
-					(reference "#PWR032")
+					(reference "#PWR038")
 					(unit 1)
 				)
@@
 		(dnp no)
 		(fields_autoplaced yes)
-		(property "Reference" "#PWR030"
+		(property "Reference" "#PWR037"
 			(at 106.68 67.31 0)
 			(effects
@@
 			(project "rp2040-programmer-calculator"
 				(path "/a76e07d4-0b9a-412a-8673-6db50899653e/0f3726b0-757f-41d2-86b9-fa06e0efb2c9"
-					(reference "#PWR030")
+					(reference "#PWR037")
 					(unit 1)
 				)
@@
 		(dnp no)
 		(fields_autoplaced yes)
-		(property "Reference" "J1"
+		(property "Reference" "J2"
 			(at 88.9 62.23 0)
 			(effects
@@
 			(project "rp2040-programmer-calculator"
 				(path "/a76e07d4-0b9a-412a-8673-6db50899653e/0f3726b0-757f-41d2-86b9-fa06e0efb2c9"
-					(reference "J1")
+					(reference "J2")
+					(unit 1)
+				)
+			)
+		)
+	)
+	(symbol
+		(lib_id "Device:R_US")
+		(at 110.49 77.47 90)
+		(unit 1)
+		(exclude_from_sim no)
+		(in_bom yes)
+		(on_board yes)
+		(dnp no)
+		(property "Reference" "R43"
+			(at 110.49 79.756 90)
+			(effects
+				(font
+					(size 1.27 1.27)
+				)
+			)
+		)
+		(property "Value" "5.1k"
+			(at 110.49 82.296 90)
+			(effects
+				(font
+					(size 1.27 1.27)
+				)
+			)
+		)
+		(property "Footprint" "Resistor_SMD:R_0603_1608Metric"
+			(at 110.744 76.454 90)
+			(effects
+				(font
+					(size 1.27 1.27)
+				)
+				(hide yes)
+			)
+		)
+		(property "Datasheet" "~"
+			(at 110.49 77.47 0)
+			(effects
+				(font
+					(size 1.27 1.27)
+				)
+				(hide yes)
+			)
+		)
+		(property "Description" "Resistor, US symbol"
+			(at 110.49 77.47 0)
+			(effects
+				(font
+					(size 1.27 1.27)
+				)
+				(hide yes)
+			)
+		)
+		(pin "2"
+		)
+		(pin "1"
+		)
+		(instances
+			(project "rp2040-programmer-calculator"
+				(path "/a76e07d4-0b9a-412a-8673-6db50899653e/0f3726b0-757f-41d2-86b9-fa06e0efb2c9"
+					(reference "R43")
 					(unit 1)
 				)
@@
 		(dnp no)
 		(fields_autoplaced yes)
-		(property "Reference" "R38"
+		(property "Reference" "R42"
 			(at 110.49 68.58 90)
 			(effects
@@
 			)
 		)
-		(property "Footprint" ""
+		(property "Footprint" "Resistor_SMD:R_0603_1608Metric"
 			(at 110.744 73.914 90)
 			(effects
@@
 			(project ""
 				(path "/a76e07d4-0b9a-412a-8673-6db50899653e/0f3726b0-757f-41d2-86b9-fa06e0efb2c9"
-					(reference "R38")
-					(unit 1)
-				)
-			)
-		)
-	)
-	(symbol
-		(lib_id "Device:R_US")
-		(at 110.49 77.47 90)
-		(unit 1)
-		(exclude_from_sim no)
-		(in_bom yes)
-		(on_board yes)
-		(dnp no)
-		(property "Reference" "R39"
-			(at 110.49 80.01 90)
-			(effects
-				(font
-					(size 1.27 1.27)
-				)
-			)
-		)
-		(property "Value" "5.1k"
-			(at 110.49 82.55 90)
-			(effects
-				(font
-					(size 1.27 1.27)
-				)
-			)
-		)
-		(property "Footprint" ""
-			(at 110.744 76.454 90)
-			(effects
-				(font
-					(size 1.27 1.27)
-				)
-				(hide yes)
-			)
-		)
-		(property "Datasheet" "~"
-			(at 110.49 77.47 0)
-			(effects
-				(font
-					(size 1.27 1.27)
-				)
-				(hide yes)
-			)
-		)
-		(property "Description" "Resistor, US symbol"
-			(at 110.49 77.47 0)
-			(effects
-				(font
-					(size 1.27 1.27)
-				)
-				(hide yes)
-			)
-		)
-		(pin "2"
-		)
-		(pin "1"
-		)
-		(instances
-			(project "rp2040-programmer-calculator"
-				(path "/a76e07d4-0b9a-412a-8673-6db50899653e/0f3726b0-757f-41d2-86b9-fa06e0efb2c9"
-					(reference "R39")
+					(reference "R42")
 					(unit 1)
 				)
@@
 		(on_board yes)
 		(dnp no)
-		(property "Reference" "#PWR031"
+		(property "Reference" "#PWR039"
 			(at 127 119.38 0)
 			(effects
@@
 			(project "rp2040-programmer-calculator"
 				(path "/a76e07d4-0b9a-412a-8673-6db50899653e/0f3726b0-757f-41d2-86b9-fa06e0efb2c9"
-					(reference "#PWR031")
-					(unit 1)
-				)
+					(reference "#PWR039")
+					(unit 1)
+				)
