File: pcb/rp2040-programmer-calculator/power.kicad_sch (KiCad schematic)
At the start: 55 parts, among them Q1 AO3401A, Q2 BSS84, Q3 MMBT3904, Q4 DMG1012T, U10 XB7608AJ, U8 TP4057, U9 TLV75533PDBV

Commit message: Finish PCB
Parts:
- removed R53, R55: 2k, Resistor_SMD:R_0603_1608Metric, symbol Device:R
- added R50, R51: 2k, Resistor_SMD:R_0603_1608Metric, symbol Device:R_US
- C10: renamed from C23; footprint Capacitor_SMD:C_0402_1005Metric -> Capacitor_SMD:C_0603_1608Metric
- C11: renamed from C24; footprint Capacitor_SMD:C_0402_1005Metric -> Capacitor_SMD:C_0603_1608Metric
- C12: renamed from C21; footprint Capacitor_SMD:C_0402_1005Metric -> Capacitor_SMD:C_0603_1608Metric
- C13: renamed from C22; footprint Capacitor_SMD:C_0402_1005Metric -> Capacitor_SMD:C_0603_1608Metric
- C14: renamed from C26; footprint Capacitor_SMD:C_0402_1005Metric -> Capacitor_SMD:C_0603_1608Metric
- C15: renamed from C25; footprint Capacitor_SMD:C_0402_1005Metric -> Capacitor_SMD:C_0603_1608Metric
- C16: renamed from C27; footprint Capacitor_SMD:C_0402_1005Metric -> Capacitor_SMD:C_0603_1608Metric
- C9: renamed from C20; footprint Capacitor_SMD:C_0402_1005Metric -> Capacitor_SMD:C_0603_1608Metric
- R44: renamed from R40; footprint (none) -> Resistor_SMD:R_0603_1608Metric
- R45: renamed from R43; footprint (none) -> Resistor_SMD:R_0603_1608Metric
- R46: renamed from R44; footprint (none) -> Resistor_SMD:R_0603_1608Metric
- R47: renamed from R50; footprint (none) -> Resistor_SMD:R_0603_1608Metric
- R48: renamed from R45; footprint (none) -> Resistor_SMD:R_0603_1608Metric
- R49: renamed from R54; footprint (none) -> Resistor_SMD:R_0603_1608Metric
- R52: renamed from R47; footprint (none) -> Resistor_SMD:R_0603_1608Metric
- R53: renamed from R46; footprint (none) -> Resistor_SMD:R_0603_1608Metric
- R54: renamed from R51; footprint (none) -> Resistor_SMD:R_0603_1608Metric
- R55: renamed from R48; footprint (none) -> Resistor_SMD:R_0603_1608Metric
- R56: renamed from R49; footprint (none) -> Resistor_SMD:R_0603_1608Metric
- R57: renamed from R52; footprint (none) -> Resistor_SMD:R_0603_1608Metric
- S1: footprint EVQP7J01P -> SamacSys_Parts:EVQP7J01P
- U10: footprint XB7608AJ:XB7608AJ -> XB7608AJ:CPC-5_L2.6-W2.6-P0.53-LS4.0-BL
- renumbered C15 to C17, C16 to C18, C9 to C19, C10 to C20, C11 to C21, C12 to C22, C13 to C23, C14 to C24, C17 to C25, C18 to C26, C19 to C27, D92 to D100, D87 to D95, D89 to D96, D90 to D97, D88 to D98, D91 to D99, TP4 to TP10, TP5 to TP11, TP6 to TP12, TP7 to TP13, TP1 to TP7, TP2 to TP8, TP3 to TP9
Connections:
- net LOAD: now also S1.2 (NO_2), R50.1, R51.1
- net at R49.1: now also S1.3 (COM_1), S1.4 (COM_2); no longer S1.2
- net at D96.2 (A): now also R50.2
- net at D97.2 (A): now also R51.2

Commit message: Finished design
Parts:
- removed S1: EVQ-P7A01P, SamacSys_Parts:EVQP7J01P, symbol SamacSys_Parts:EVQ-P7A01P
- added SW65: EVQ-P7A01P, EVQP7J01P:EVQP7J01P, symbol Switch:SW_Push
- BT1: footprint Connector_JST:JST_PH_S2B-PH-K_1x02_P2.00mm_Horizontal_Reverse_Polarity -> JST_PH_S2B_Reverse_Polarity:JST_PH_S2B-PH-K_1x02_P2.00mm_Horizontal
- C15: value 0.1u -> 100n
Connections:
- net LOAD: now also SW65.1
- net at R49.1: now also SW65.2

Commit message: Add RP2040 project
Parts:
- removed SW65: EVQ-P7A01P, EVQP7J01P:EVQP7J01P, symbol Switch:SW_Push
- added SW64: HX TS24CA, HX-TS24CA:HX-TS24CA, symbol Switch:SW_Push
Connections:
- net LOAD: now also SW64.2
- net at R49.1: now also SW64.1
Changed lines of the file:
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@@
+	)
+	(symbol
+		(lib_id "Switch:SW_Push")
+		(at 242.57 107.95 0)
+		(mirror y)
+		(unit 1)
+		(exclude_from_sim no)
+		(in_bom yes)
+		(on_board yes)
+		(dnp no)
+		(property "Reference" "SW64"
+			(at 242.57 100.33 0)
+			(effects
+				(font
+					(size 1.27 1.27)
+				)
+			)
+		)
+		(property "Value" "HX TS24CA"
+			(at 242.57 102.87 0)
+			(effects
+				(font
+					(size 1.27 1.27)
+				)
+			)
+		)
+		(property "Footprint" "HX-TS24CA:HX-TS24CA"
+			(at 242.57 102.87 0)
+			(effects
+				(font
+					(size 1.27 1.27)
+				)
+				(hide yes)
+			)
+		)
+		(property "Datasheet" "~"
+			(at 242.57 102.87 0)
+			(effects
+				(font
+					(size 1.27 1.27)
+				)
+				(hide yes)
+			)
+		)
+		(property "Description" "Push button switch, generic, two pins"
+			(at 242.57 107.95 0)
+			(effects
+				(font
+					(size 1.27 1.27)
+				)
+				(hide yes)
+			)
+		)
+		(pin "1"
+		)
+		(pin "2"
+		)
+		(instances
+			(project ""
+				(path "/a76e07d4-0b9a-412a-8673-6db50899653e/98749e6e-b27c-4355-8130-c67da41bd9d3"
+					(reference "SW64")
+					(unit 1)
+				)
+			)
+		)
 	)
 	(symbol
@@
 					(unit 1)
 				)
-			)
-		)
-	)
-	(symbol
-		(lib_id "Switch:SW_Push")
-		(at 242.57 107.95 0)
-		(unit 1)
-		(exclude_from_sim no)
-		(in_bom yes)
-		(on_board yes)
-		(dnp no)
-		(fields_autoplaced yes)
-		(property "Reference" "SW65"
-			(at 242.57 100.33 0)
-			(effects
-				(font
-					(size 1.27 1.27)
-				)
-			)
-		)
-		(property "Value" "EVQ-P7A01P"
-			(at 242.57 102.87 0)
-			(effects
-				(font
-					(size 1.27 1.27)
-				)
-			)
-		)
-		(property "Footprint" "EVQP7J01P:EVQP7J01P"
-			(at 242.57 102.87 0)
-			(effects
-				(font
-					(size 1.27 1.27)
-				)
-				(hide yes)
-			)
-		)
-		(property "Datasheet" "https://industrial.panasonic.com/cdbs/www-data/pdf/ATK0000/ATK0000C378.pdf"
-			(at 242.57 102.87 0)
-			(effects
-				(font
-					(size 1.27 1.27)
-				)
-				(hide yes)
-			)
-		)
-		(property "Description" "Black Side Tactile Switch, Single Pole Single Throw (SPST) 50 mA @ 12 V dc 1.7mm"
-			(at 242.57 107.95 0)
-			(effects
-				(font
-					(size 1.27 1.27)
-				)
-				(hide yes)
-			)
-		)
-		(pin "1"
-		)
-		(pin "2"
-		)
-		(instances
-			(project ""
-				(path "/a76e07d4-0b9a-412a-8673-6db50899653e/98749e6e-b27c-4355-8130-c67da41bd9d3"
-					(reference "SW65")
-					(unit 1)
-				)
